Commit message: Update-2

File: src/my_robot_description/urdf/camera.xacro (robot description, xacro)
@@ -23,4 +23,10 @@
     <child link="camera_link" />
     <origin xyz="${(base_length + camera_length)/2.0} 0 ${base_height/2.0}" rpy="0 0 0"/>
+</joint>
+<link name="camera_link_optical" />
+<joint name="camera_optical_joint" type="fixed">
+    <origin xyz="0 0 0" rpy="${-pi/2} 0 ${-pi/2}"/>
+    <parent link="camera_link"/>
+    <child link="camera_link_optical"/>
 </joint>
 <gazebo reference="camera_link">

File: src/my_robot_description/urdf/common_properties.urdf.xacro (robot description, xacro)
@@ -15,4 +15,13 @@
     <material name="black">
         <color rgba="0.0 0.0 0.0 1.0" />
+    </material>
+    <material name="color_1">
+        <color rgba="0.941 0.573 0.804 1.0" />
+    </material>
+    <material name="color_2">
+        <color rgba="0.800 0.267 0.294 1.0" />
+    </material>
+    <material name="color_3">
+        <color rgba="0.957 0.910 0.757 1.0" />
     </material>
     <xacro:macro name="box_inertia" params="m x y z o_xyz o_rpy">

File: src/my_robot_description/urdf/my_robot.urdf.xacro (robot description, xacro)
@@ -4,4 +4,11 @@
     <xacro:include filename="mobile_base.urdf.xacro" />
     <xacro:include filename="mobile_base_gazebo.urdf.xacro" />
+    <xacro:include filename="arm.xacro" />
+    <xacro:include filename="arm_gazebo.xacro" />
     <xacro:include filename="camera.xacro" />
+    <joint name="mobile_base_arm_joint" type="fixed">
+        <parent link="base_link" />
+        <child link="arm_base_link" />
+        <origin xyz="${base_length / 4.0} 0 ${base_height}" rpy="0 0 0"/>
+    </joint>
 </robot>
